Commit message: .

File: src/receptionist_robot_description/urdf/receptionist_robot.urdf.xacro (robot description, xacro)
@@ -28,8 +28,8 @@
   <!-- Lidar mount offsets -->
   <!-- Placed near the front edge of the robot and elevated on a mast or shelf -->
-  <xacro:property name="lidar_offset_x" value="0.24" />
+  <xacro:property name="lidar_offset_x" value="0.0" />
   <xacro:property name="lidar_offset_y" value="0.0" />
   <xacro:property name="lidar_offset_z" value="0.25" />
-  <xacro:property name="lidar_mass" value="0.12" />
+  <xacro:property name="lidar_mass" value="0.25" />
   <!-- ==================================================================== -->
   <!-- MATERIALS (Colors for visualization in RViz)                         -->

Commit message: Add robot_localization EKF node and imu_link frame for MPU9250 sensor fusion

File: src/receptionist_robot_description/urdf/receptionist_robot.urdf.xacro (robot description, xacro)
@@ -228,3 +228,18 @@
     <origin xyz="${lidar_offset_x} ${lidar_offset_y} ${lidar_offset_z}" rpy="0 0 0" />
   </joint>
+  <!-- 9. IMU Sensor (frame_id = imu_link) -->
+  <link name="imu_link">
+    <visual>
+      <origin xyz="0 0 0" rpy="0 0 0" />
+      <geometry>
+        <box size="0.02 0.02 0.005" />
+      </geometry>
+      <material name="lidar_material" />
+    </visual>
+  </link>
+  <joint name="imu_joint" type="fixed">
+    <parent link="base_link" />
+    <child link="imu_link" />
+    <origin xyz="0.0 0.0 0.10" rpy="0 0 0" />
+  </joint>
 </robot>

Commit message: update odom with ekf

File: src/receptionist_robot_description/urdf/receptionist_robot.urdf.xacro (robot description, xacro)
@@ -6,9 +6,9 @@
   <!-- Wheel specifications -->
   <!-- Wheel diameter: 0.065m (6.5cm), radius: 0.0325m -->
-  <xacro:property name="wheel_radius" value="0.0325" />
+  <xacro:property name="wheel_radius" value="0.04" />
   <!-- Wheel width (thickness): 0.025m (2.5cm) -->
-  <xacro:property name="wheel_width" value="0.03" />
+  <xacro:property name="wheel_width" value="0.02" />
   <!-- Wheelbase: 0.30m (30.0cm) separation between wheels along Y-axis -->
-  <xacro:property name="wheelbase" value="0.30" />
+  <xacro:property name="wheelbase" value="0.395" />
   <!-- Wheel mass: 0.15kg -->
   <xacro:property name="wheel_mass" value="0.15" />
@@ -17,5 +17,5 @@
   <xacro:property name="chassis_radius" value="0.18" />
   <xacro:property name="chassis_height" value="0.50" />
-  <xacro:property name="chassis_mass" value="10.0" />
+  <xacro:property name="chassis_mass" value="20.0" />
   <!-- Caster specifications -->
   <!-- Sphere caster diameter is sized to touch the ground.

Commit message: save commit

File: src/receptionist_robot_description/urdf/receptionist_robot.urdf.xacro (robot description, xacro)
@@ -28,7 +28,7 @@
   <!-- Lidar mount offsets -->
   <!-- Placed near the front edge of the robot and elevated on a mast or shelf -->
-  <xacro:property name="lidar_offset_x" value="0.0" />
+  <xacro:property name="lidar_offset_x" value="-0.01" />
   <xacro:property name="lidar_offset_y" value="0.0" />
-  <xacro:property name="lidar_offset_z" value="0.25" />
+  <xacro:property name="lidar_offset_z" value="0.17" />
   <xacro:property name="lidar_mass" value="0.25" />
   <!-- ==================================================================== -->
@@ -208,5 +208,5 @@
   <link name="laser">
     <visual>
-      <origin xyz="0 0 0" rpy="0 0 0" />
+      <origin xyz="-0.1 0 0.17" rpy="0 0 0" />
       <geometry>
         <!-- Standard puck cylinder shape for RPLidar A1/A2 -->
@@ -231,5 +231,5 @@
   <link name="imu_link">
     <visual>
-      <origin xyz="0 0 0" rpy="0 0 0" />
+      <origin xyz="0.01 0 0.1" rpy="0 0 0" />
       <geometry>
         <box size="0.02 0.02 0.005" />
@@ -241,5 +241,5 @@
     <parent link="base_link" />
     <child link="imu_link" />
-    <origin xyz="0.0 0.0 0.10" rpy="0 0 0" />
+    <origin xyz="0.01 0.0 0.10" rpy="0 0 0" />
   </joint>
 </robot>

Commit message: Update receptionist robot packages, kiosk scripts, and configurations; remove large media files and build artifacts

File: src/receptionist_robot_description/urdf/receptionist_robot.urdf.xacro (robot description, xacro)
@@ -30,5 +30,5 @@
   <xacro:property name="lidar_offset_x" value="-0.01" />
   <xacro:property name="lidar_offset_y" value="0.0" />
-  <xacro:property name="lidar_offset_z" value="0.17" />
+  <xacro:property name="lidar_offset_z" value="0.16" />
   <xacro:property name="lidar_mass" value="0.25" />
   <!-- ==================================================================== -->
@@ -243,3 +243,24 @@
     <origin xyz="0.01 0.0 0.10" rpy="0 0 0" />
   </joint>
+  <!-- 10. USB Camera (frame_id = camera_link & camera_color_optical_frame) -->
+  <link name="camera_link">
+    <visual>
+      <origin xyz="0 0 0" rpy="0 0 0" />
+      <geometry>
+        <box size="0.03 0.08 0.03" />
+      </geometry>
+      <material name="lidar_material" />
+    </visual>
+  </link>
+  <joint name="camera_joint" type="fixed">
+    <parent link="base_link" />
+    <child link="camera_link" />
+    <origin xyz="-0.06 0.0 1.16" rpy="0 0 0" />
+  </joint>
+  <link name="camera_color_optical_frame" />
+  <joint name="camera_optical_joint" type="fixed">
+    <parent link="camera_link" />
+    <child link="camera_color_optical_frame" />
+    <origin xyz="0 0 0" rpy="${-pi/2} 0 ${-pi/2}" />
+  </joint>
 </robot>

Commit message: 22-8-2026:2

File: src/receptionist_robot_description/urdf/receptionist_robot.urdf.xacro (robot description, xacro)
@@ -26,10 +26,33 @@
   <xacro:property name="caster_offset_x" value="0.12" />
   <xacro:property name="caster_mass" value="0.2" />
-  <!-- Lidar mount offsets -->
-  <!-- Placed near the front edge of the robot and elevated on a mast or shelf -->
-  <xacro:property name="lidar_offset_x" value="-0.01" />
-  <xacro:property name="lidar_offset_y" value="0.0" />
-  <xacro:property name="lidar_offset_z" value="0.16" />
+  <!-- ==================================================================== -->
+  <!-- SENSOR MOUNTING COORDINATES & OFFSETS (LiDAR, IMU, CAMERA)          -->
+  <!-- ==================================================================== -->
+  <!-- ROS COORDINATE CONVENTION (REP-103):
+       Coordinate Origin (0, 0, 0) is "base_link" = MIDPOINT OF THE WHEEL AXLE.
+       - X axis (meters): Positive (+) = FORWARD | Negative (-) = BACKWARD
+       - Y axis (meters): Positive (+) = LEFT    | Negative (-) = RIGHT
+       - Z axis (meters): Positive (+) = UP      | Negative (-) = DOWN
+       - Rotation rpy (radians):
+           * roll  : Rotation about X-axis (tilt left/right)
+           * pitch : Rotation about Y-axis (tilt nose up/down)
+           * yaw   : Rotation about Z-axis (heading / turning left/right).
+                     0 = Facing forward; pi (3.14159) = Facing backwards;
+                     pi/2 (1.5708) = Facing left; -pi/2 (-1.5708) = Facing right.
+  -->
+  <!-- 1. LiDAR Sensor Offsets (Laser Scanner) -->
+  <!-- Physical offset measured from wheel axle center to LiDAR scanning center -->
+  <xacro:property name="lidar_offset_x" value="0.0" /> <!-- meters: Forward (+) or Backward (-) from wheel axle center -->
+  <xacro:property name="lidar_offset_y" value="0.0" />  <!-- meters: Left (+) or Right (-) -->
+  <xacro:property name="lidar_offset_z" value="0.16" /> <!-- meters: Height from wheel axle center to LiDAR scan plane -->
+  <xacro:property name="lidar_offset_yaw" value="0.0" /><!-- radians: Yaw rotation (e.g. 3.14159 if mounted facing backwards) -->
   <xacro:property name="lidar_mass" value="0.25" />
+  <!-- 2. IMU Sensor Offsets (Inertial Measurement Unit) -->
+  <!-- Physical position of IMU chip relative to wheel axle center -->
+  <xacro:property name="imu_offset_x" value="0.0" /> <!-- meters: IMU position along X axis -->
+  <xacro:property name="imu_offset_y" value="0.0" />  <!-- meters: IMU position along Y axis -->
+  <xacro:property name="imu_offset_z" value="0.10" /> <!-- meters: Height of IMU along Z axis -->
+  <xacro:property name="imu_offset_yaw" value="0.0" /><!-- radians: Mounting yaw orientation of IMU -->
+  <!-- ==================================================================== -->
   <!-- ==================================================================== -->
   <!-- MATERIALS (Colors for visualization in RViz)                         -->
@@ -205,10 +228,15 @@
     <origin xyz="-${caster_offset_x} 0 ${-(wheel_radius - caster_radius)}" rpy="0 0 0" />
   </joint>
-  <!-- 8. Lidar Sensor (frame_id = laser) -->
+  <!-- ==================================================================== -->
+  <!-- 8. Lidar Sensor (frame_id = laser)                                   -->
+  <!-- ==================================================================== -->
+  <!-- LINK "laser": 2D laser scanner sensor link.
+       NOTE: Origin for visual & collision is set to (0,0,0) so the geometry center
+       matches the measurement origin of frame "laser". -->
   <link name="laser">
     <visual>
-      <origin xyz="-0.1 0 0.17" rpy="0 0 0" />
-      <geometry>
-        <!-- Standard puck cylinder shape for RPLidar A1/A2 -->
+      <origin xyz="0 0 0" rpy="0 0 0" />
+      <geometry>
+        <!-- Cylindrical puck representing LiDAR sensor (HCLiDAR / RPLidar) -->
         <cylinder radius="0.035" length="0.04" />
       </geometry>
@@ -223,13 +251,21 @@
     <xacro:cylinder_inertia mass="${lidar_mass}" r="0.035" h="0.04" />
   </link>
+  <!-- JOINT "laser_joint": Fixed transform between base_link and laser frame.
+       Critical for SLAM scan matching and Nav2 costmap obstacle placement.
+       - origin xyz: [x = forward(+)/backward(-), y = left(+)/right(-), z = up(+)/down(-)]
+       - origin rpy: [roll, pitch, yaw] (yaw = pi if mounted facing backward)
+       (Easily tuned via <xacro:property name="lidar_offset_..."/> at the top of this file) -->
   <joint name="laser_joint" type="fixed">
     <parent link="base_link" />
     <child link="laser" />
-    <origin xyz="${lidar_offset_x} ${lidar_offset_y} ${lidar_offset_z}" rpy="0 0 0" />
-  </joint>
-  <!-- 9. IMU Sensor (frame_id = imu_link) -->
+    <origin xyz="${lidar_offset_x} ${lidar_offset_y} ${lidar_offset_z}" rpy="0 0 ${lidar_offset_yaw}" />
+  </joint>
+  <!-- ==================================================================== -->
+  <!-- 9. IMU Sensor (frame_id = imu_link)                                  -->
+  <!-- ==================================================================== -->
+  <!-- LINK "imu_link": 6-DOF / 9-DOF inertial measurement unit module -->
   <link name="imu_link">
     <visual>
-      <origin xyz="0.01 0 0.1" rpy="0 0 0" />
+      <origin xyz="0 0 0" rpy="0 0 0" />
       <geometry>
         <box size="0.02 0.02 0.005" />
@@ -238,8 +274,11 @@
     </visual>
   </link>
+  <!-- JOINT "imu_joint": Fixed transform between base_link and imu_link.
+       Used by EKF (robot_localization) to fuse angular velocity and linear acceleration.
+       (Easily tuned via <xacro:property name="imu_offset_..."/> at the top of this file) -->
   <joint name="imu_joint" type="fixed">
     <parent link="base_link" />
     <child link="imu_link" />
-    <origin xyz="0.01 0.0 0.10" rpy="0 0 0" />
+    <origin xyz="${imu_offset_x} ${imu_offset_y} ${imu_offset_z}" rpy="0 0 ${imu_offset_yaw}" />
   </joint>
   <!-- 10. USB Camera (frame_id = camera_link & camera_color_optical_frame) -->

Commit message: 27-8-2026/1

File: src/receptionist_robot_description/urdf/receptionist_robot.urdf.xacro (robot description, xacro)
@@ -28,5 +28,5 @@
   <!-- Lidar mount offsets -->
   <!-- Placed near the front edge of the robot and elevated on a mast or shelf -->
-  <xacro:property name="lidar_offset_x" value="-0.01" />
+  <xacro:property name="lidar_offset_x" value="0.0" />
   <xacro:property name="lidar_offset_y" value="0.0" />
   <xacro:property name="lidar_offset_z" value="0.16" />
@@ -231,5 +231,5 @@
   <link name="imu_link">
     <visual>
-      <origin xyz="0.01 0 0.1" rpy="0 0 0" />
+      <origin xyz="0.0 0.0 0.1" rpy="0 0 0" />
       <geometry>
         <box size="0.02 0.02 0.005" />
@@ -241,5 +241,5 @@
     <parent link="base_link" />
     <child link="imu_link" />
-    <origin xyz="0.01 0.0 0.10" rpy="0 0 0" />
+    <origin xyz="0.0 0.0 0.10" rpy="0 0 0" />
   </joint>
   <!-- 10. USB Camera (frame_id = camera_link & camera_color_optical_frame) -->
